File: atmega328/Precision Arduino Charlieplex.kicad_pcb (KiCad board)
At the start: 2 copper layers, 76.2 x 76.2 mm, 155 parts, among them J1 M04PTH, J2 M04PTH, J3 M06SIP, J402 EM406, J403 M06SIP, J404 EM406, J405 M081X08, J406 M081X08, J5 M06SIP, U401 ATMEGA328, U501 FT232RLSSOP, U601 ZF7, U602 ZF7, U603 ZF7, Y401 12.00

Commit message: Updated to Precision 1.1 (the operational version)
Parts:
- removed J402, J404: EM406, Precision Arduino Charlieplex:EM406
- removed J403: M06SIP, Precision Arduino Charlieplex:1X06
- removed U601, U603: ZF7, Precision Arduino Charlieplex:SC-70-6
- added D200: GREEN, Precision Arduino Charlieplex 1.1:LED-0603, F.Cu at (105.3, 143.1)
- added D201: GREEN, Precision Arduino Charlieplex 1.1:LED-0603, F.Cu at (100.2, 143.1)
- added D202: GREEN, Precision Arduino Charlieplex 1.1:LED-0603, F.Cu at (95.2, 143.1)
- added D203: GREEN, Precision Arduino Charlieplex 1.1:LED-0603, F.Cu at (90.1, 143.1)
- added D204: GREEN, Precision Arduino Charlieplex 1.1:LED-0603, F.Cu at (85.0, 143.1)
- added D205: GREEN, Precision Arduino Charlieplex 1.1:LED-0603, F.Cu at (79.9, 143.1)
- added D206: GREEN, Precision Arduino Charlieplex 1.1:LED-0603, F.Cu at (74.8, 143.1)
- added D207: GREEN, Precision Arduino Charlieplex 1.1:LED-0603, F.Cu at (69.8, 143.1)
- added D208: GREEN, Precision Arduino Charlieplex 1.1:LED-0603, F.Cu at (64.7, 143.1)
- added D209: GREEN, Precision Arduino Charlieplex 1.1:LED-0603, F.Cu at (59.6, 143.1)
- added D210: GREEN, Precision Arduino Charlieplex 1.1:LED-0603, F.Cu at (54.5, 143.1)
- added D211: GREEN, Precision Arduino Charlieplex 1.1:LED-0603, F.Cu at (49.4, 143.1)
- added D212: GREEN, Precision Arduino Charlieplex 1.1:LED-0603, F.Cu at (44.4, 143.1)
- added D213: GREEN, Precision Arduino Charlieplex 1.1:LED-0603, F.Cu at (39.3, 143.1)
- added D214: GREEN, Precision Arduino Charlieplex 1.1:LED-0603, F.Cu at (34.2, 143.1)
- added D215: GREEN, Precision Arduino Charlieplex 1.1:LED-0603, F.Cu at (29.1, 143.1)
- added D216: GREEN, Precision Arduino Charlieplex 1.1:LED-0603, F.Cu at (24.0, 143.1)
- added D217: GREEN, Precision Arduino Charlieplex 1.1:LED-0603, F.Cu at (19.0, 143.1)
- added D218: GREEN, Precision Arduino Charlieplex 1.1:LED-0603, F.Cu at (13.9, 143.1)
- added D219: GREEN, Precision Arduino Charlieplex 1.1:LED-0603, F.Cu at (8.80, 143.1)
- added D220: GREEN, Precision Arduino Charlieplex 1.1:LED-0603, F.Cu at (3.72, 143.1)
- added D221: GREEN, Precision Arduino Charlieplex 1.1:LED-0603, F.Cu at (-1.36, 143.1)
- added D222: GREEN, Precision Arduino Charlieplex 1.1:LED-0603, F.Cu at (-6.44, 143.1)
- added D223: GREEN, Precision Arduino Charlieplex 1.1:LED-0603, F.Cu at (-11.5, 143.1)
- added D224: GREEN, Precision Arduino Charlieplex 1.1:LED-0603, F.Cu at (-16.6, 143.1)
- added D225: GREEN, Precision Arduino Charlieplex 1.1:LED-0603, F.Cu at (-21.7, 143.1)
- added D226: GREEN, Precision Arduino Charlieplex 1.1:LED-0603, F.Cu at (-26.8, 143.1)
- added D227: GREEN, Precision Arduino Charlieplex 1.1:LED-0603, F.Cu at (-31.8, 143.1)
- added D228: GREEN, Precision Arduino Charlieplex 1.1:LED-0603, F.Cu at (-36.9, 143.1)
- added D229: GREEN, Precision Arduino Charlieplex 1.1:LED-0603, F.Cu at (-42.0, 143.1)
- added D230: GREEN, Precision Arduino Charlieplex 1.1:LED-0603, F.Cu at (-47.1, 143.1)
- added D231: GREEN, Precision Arduino Charlieplex 1.1:LED-0603, F.Cu at (-52.2, 143.1)
- added D232: GREEN, Precision Arduino Charlieplex 1.1:LED-0603, F.Cu at (-57.2, 143.1)
- added D233: GREEN, Precision Arduino Charlieplex 1.1:LED-0603, F.Cu at (-62.3, 143.1)
- added D234: GREEN, Precision Arduino Charlieplex 1.1:LED-0603, F.Cu at (-67.4, 143.1)
- added D235: GREEN, Precision Arduino Charlieplex 1.1:LED-0603, F.Cu at (-72.5, 143.1)
- added D236: GREEN, Precision Arduino Charlieplex 1.1:LED-0603, F.Cu at (-77.6, 143.1)
- added D237: GREEN, Precision Arduino Charlieplex 1.1:LED-0603, F.Cu at (-82.6, 143.1)
- added D238: GREEN, Precision Arduino Charlieplex 1.1:LED-0603, F.Cu at (-87.7, 143.1)
- added D239: GREEN, Precision Arduino Charlieplex 1.1:LED-0603, F.Cu at (-92.8, 143.1)
- added D240: GREEN, Precision Arduino Charlieplex 1.1:LED-0603, F.Cu at (-97.9, 143.1)
- added D241: GREEN, Precision Arduino Charlieplex 1.1:LED-0603, F.Cu at (-103.0, 143.1)
- added D242: GREEN, Precision Arduino Charlieplex 1.1:LED-0603, F.Cu at (-108.0, 143.1)
- added D243: GREEN, Precision Arduino Charlieplex 1.1:LED-0603, F.Cu at (-113.1, 143.1)
- added D244: GREEN, Precision Arduino Charlieplex 1.1:LED-0603, F.Cu at (-118.2, 143.1)
- added D245: GREEN, Precision Arduino Charlieplex 1.1:LED-0603, F.Cu at (-123.3, 143.1)
- added D246: GREEN, Precision Arduino Charlieplex 1.1:LED-0603, F.Cu at (-128.4, 143.1)
- added D247: GREEN, Precision Arduino Charlieplex 1.1:LED-0603, F.Cu at (-133.4, 143.1)
- added D248: GREEN, Precision Arduino Charlieplex 1.1:LED-0603, F.Cu at (-138.5, 143.1)
- added D249: GREEN, Precision Arduino Charlieplex 1.1:LED-0603, F.Cu at (-143.6, 143.1)
- added D250: GREEN, Precision Arduino Charlieplex 1.1:LED-0603, F.Cu at (-148.7, 143.1)
- added D251: GREEN, Precision Arduino Charlieplex 1.1:LED-0603, F.Cu at (-153.8, 143.1)
- added D252: GREEN, Precision Arduino Charlieplex 1.1:LED-0603, F.Cu at (-158.8, 143.1)
- added D253: GREEN, Precision Arduino Charlieplex 1.1:LED-0603, F.Cu at (-163.9, 143.1)
- added D254: GREEN, Precision Arduino Charlieplex 1.1:LED-0603, F.Cu at (-169.0, 143.1)
- added D255: GREEN, Precision Arduino Charlieplex 1.1:LED-0603, F.Cu at (-174.1, 143.1)
- added D256: GREEN, Precision Arduino Charlieplex 1.1:LED-0603, F.Cu at (-179.2, 143.1)
- added D257: GREEN, Precision Arduino Charlieplex 1.1:LED-0603, F.Cu at (-184.2, 143.1)
- added D258: GREEN, Precision Arduino Charlieplex 1.1:LED-0603, F.Cu at (-189.3, 143.1)
- added D259: GREEN, Precision Arduino Charlieplex 1.1:LED-0603, F.Cu at (-194.4, 143.1)
- added D300: BLUE, Precision Arduino Charlieplex 1.1:LED-0603, F.Cu at (-199.5, 143.1)
- added D301: BLUE, Precision Arduino Charlieplex 1.1:LED-0603, F.Cu at (-204.6, 143.1)
- added D302: BLUE, Precision Arduino Charlieplex 1.1:LED-0603, F.Cu at (-209.6, 143.1)
- added D303: BLUE, Precision Arduino Charlieplex 1.1:LED-0603, F.Cu at (-214.7, 143.1)
- added D304: BLUE, Precision Arduino Charlieplex 1.1:LED-0603, F.Cu at (-219.8, 143.1)
- added D305: BLUE, Precision Arduino Charlieplex 1.1:LED-0603, F.Cu at (-224.9, 143.1)
- added D306: BLUE, Precision Arduino Charlieplex 1.1:LED-0603, F.Cu at (-230.0, 143.1)
- added D307: BLUE, Precision Arduino Charlieplex 1.1:LED-0603, F.Cu at (-235.0, 143.1)
- added D308: BLUE, Precision Arduino Charlieplex 1.1:LED-0603, F.Cu at (-240.1, 143.1)
- added D309: BLUE, Precision Arduino Charlieplex 1.1:LED-0603, F.Cu at (-245.2, 143.1)
- added D310: BLUE, Precision Arduino Charlieplex 1.1:LED-0603, F.Cu at (-250.3, 143.1)
- added D311: BLUE, Precision Arduino Charlieplex 1.1:LED-0603, F.Cu at (-255.4, 143.1)
- added D312: BLUE, Precision Arduino Charlieplex 1.1:LED-0603, F.Cu at (-260.4, 143.1)
- added D313: BLUE, Precision Arduino Charlieplex 1.1:LED-0603, F.Cu at (-265.5, 143.1)
- added D314: BLUE, Precision Arduino Charlieplex 1.1:LED-0603, F.Cu at (-270.6, 143.1)
- added D315: BLUE, Precision Arduino Charlieplex 1.1:LED-0603, F.Cu at (-275.7, 143.1)
- added D316: BLUE, Precision Arduino Charlieplex 1.1:LED-0603, F.Cu at (-280.8, 143.1)
- added D317: BLUE, Precision Arduino Charlieplex 1.1:LED-0603, F.Cu at (-285.8, 143.1)
- added D318: BLUE, Precision Arduino Charlieplex 1.1:LED-0603, F.Cu at (-290.9, 143.1)
- added D319: BLUE, Precision Arduino Charlieplex 1.1:LED-0603, F.Cu at (-296.0, 143.1)
- added D320: BLUE, Precision Arduino Charlieplex 1.1:LED-0603, F.Cu at (-301.1, 143.1)
- added D321: BLUE, Precision Arduino Charlieplex 1.1:LED-0603, F.Cu at (-306.2, 143.1)
- added D322: BLUE, Precision Arduino Charlieplex 1.1:LED-0603, F.Cu at (-311.2, 143.1)
- added D323: BLUE, Precision Arduino Charlieplex 1.1:LED-0603, F.Cu at (-316.3, 143.1)
- added D324: BLUE, Precision Arduino Charlieplex 1.1:LED-0603, F.Cu at (-321.4, 143.1)
- added D325: BLUE, Precision Arduino Charlieplex 1.1:LED-0603, F.Cu at (-326.5, 143.1)
- added D326: BLUE, Precision Arduino Charlieplex 1.1:LED-0603, F.Cu at (-331.6, 143.1)
- added D327: BLUE, Precision Arduino Charlieplex 1.1:LED-0603, F.Cu at (-336.6, 143.1)
- added D328: BLUE, Precision Arduino Charlieplex 1.1:LED-0603, F.Cu at (-341.7, 143.1)
- added D329: BLUE, Precision Arduino Charlieplex 1.1:LED-0603, F.Cu at (-346.8, 143.1)
- added D330: BLUE, Precision Arduino Charlieplex 1.1:LED-0603, F.Cu at (-351.9, 143.1)
- added D331: BLUE, Precision Arduino Charlieplex 1.1:LED-0603, F.Cu at (-357.0, 143.1)
- added D332: BLUE, Precision Arduino Charlieplex 1.1:LED-0603, F.Cu at (-362.0, 143.1)
- added D333: BLUE, Precision Arduino Charlieplex 1.1:LED-0603, F.Cu at (-367.1, 143.1)
- added D334: BLUE, Precision Arduino Charlieplex 1.1:LED-0603, F.Cu at (-372.2, 143.1)
- added D335: BLUE, Precision Arduino Charlieplex 1.1:LED-0603, F.Cu at (-377.3, 143.1)
- added D336: BLUE, Precision Arduino Charlieplex 1.1:LED-0603, F.Cu at (-382.4, 143.1)
- added D337: BLUE, Precision Arduino Charlieplex 1.1:LED-0603, F.Cu at (-387.4, 143.1)
- added D338: BLUE, Precision Arduino Charlieplex 1.1:LED-0603, F.Cu at (-392.5, 143.1)
- added D339: BLUE, Precision Arduino Charlieplex 1.1:LED-0603, F.Cu at (-397.6, 143.1)
- added D340: BLUE, Precision Arduino Charlieplex 1.1:LED-0603, F.Cu at (-402.7, 143.1)
- added D341: BLUE, Precision Arduino Charlieplex 1.1:LED-0603, F.Cu at (-407.8, 143.1)
- added D342: BLUE, Precision Arduino Charlieplex 1.1:LED-0603, F.Cu at (-412.8, 143.1)
- added D343: BLUE, Precision Arduino Charlieplex 1.1:LED-0603, F.Cu at (-417.9, 143.1)
- added D344: BLUE, Precision Arduino Charlieplex 1.1:LED-0603, F.Cu at (-423.0, 143.1)
- added D345: BLUE, Precision Arduino Charlieplex 1.1:LED-0603, F.Cu at (-428.1, 143.1)
- added D346: BLUE, Precision Arduino Charlieplex 1.1:LED-0603, F.Cu at (-433.2, 143.1)
- added D347: BLUE, Precision Arduino Charlieplex 1.1:LED-0603, F.Cu at (-438.2, 143.1)
- added D348: BLUE, Precision Arduino Charlieplex 1.1:LED-0603, F.Cu at (-443.3, 143.1)
- added D349: BLUE, Precision Arduino Charlieplex 1.1:LED-0603, F.Cu at (-448.4, 143.1)
- added D350: BLUE, Precision Arduino Charlieplex 1.1:LED-0603, F.Cu at (-453.5, 143.1)
- added D351: BLUE, Precision Arduino Charlieplex 1.1:LED-0603, F.Cu at (-458.6, 143.1)
- added D352: BLUE, Precision Arduino Charlieplex 1.1:LED-0603, F.Cu at (-463.6, 143.1)
- added D353: BLUE, Precision Arduino Charlieplex 1.1:LED-0603, F.Cu at (-468.7, 143.1)
- added D354: BLUE, Precision Arduino Charlieplex 1.1:LED-0603, F.Cu at (-473.8, 143.1)
- added D355: BLUE, Precision Arduino Charlieplex 1.1:LED-0603, F.Cu at (-478.9, 143.1)
- added D356: BLUE, Precision Arduino Charlieplex 1.1:LED-0603, F.Cu at (-484.0, 143.1)
- added D357: BLUE, Precision Arduino Charlieplex 1.1:LED-0603, F.Cu at (-489.0, 143.1)
- added D358: BLUE, Precision Arduino Charlieplex 1.1:LED-0603, F.Cu at (-494.1, 143.1)
- added D359: BLUE, Precision Arduino Charlieplex 1.1:LED-0603, F.Cu at (-499.2, 143.1)
- added J4: M04PTH, Precision Arduino Charlieplex 1.1:1X04, F.Cu at (161.2, 98.7)
- added JP5: M02PTH, Precision Arduino Charlieplex 1.1:1X02, F.Cu at (161.2, 108.8)
- C10, C407, C408, C418, C420, C502: footprint Precision Arduino Charlieplex:0603-CAP -> Precision Arduino Charlieplex 1.1:0603-CAP
- D0, D1, D10, D11, D12, D13, D14, D15, D16, D17, D18, D19, D2, D20, D21, D22, D23, D24, D25, D26, D27, D28, D29, D3, D30, D31, D32, D33, D34, D35, D36, D37, D38, D39, D4, D40, D41, D42, D43, D44, D45, D46, D47, D48, D49, D5, D50, D51, D52, D53, D54, D55, D56, D57, D58, D59, D6, D7, D8, D9: value HOUR -> RED; footprint Precision Arduino Charlieplex:LED-0603 -> Precision Arduino Charlieplex 1.1:LED-0603
- D100, D101, D102, D103, D104, D105, D106, D107, D108, D109, D110, D111, D112, D113, D114, D115, D116, D117, D118, D119, D120, D121, D122, D123, D124, D125, D126, D127, D128, D129, D130, D131, D132, D133, D134, D135, D136, D137, D138, D139, D140, D141, D142, D143, D144, D145, D146, D147, D148, D149, D150, D151, D152, D153, D154, D155, D156, D157, D158, D159: value HOUR -> YELLOW; footprint Precision Arduino Charlieplex:LED-0603 -> Precision Arduino Charlieplex 1.1:LED-0603
- D501: value LED0603 -> BLUE; footprint Precision Arduino Charlieplex:LED-0603 -> Precision Arduino Charlieplex 1.1:LED-0603
- D502: value LED0603 -> RED; footprint Precision Arduino Charlieplex:LED-0603 -> Precision Arduino Charlieplex 1.1:LED-0603
- J1, J2: footprint Precision Arduino Charlieplex:1X04 -> Precision Arduino Charlieplex 1.1:1X04
- J3, J5: footprint Precision Arduino Charlieplex:1X06 -> Precision Arduino Charlieplex 1.1:1X06
- J405, J406: footprint Precision Arduino Charlieplex:1X08 -> Precision Arduino Charlieplex 1.1:1X08
- JP1, JP2, JP3, JP4: footprint Precision Arduino Charlieplex:STAND-OFF -> Precision Arduino Charlieplex 1.1:STAND-OFF
- R1, R2, R3, R4, R606: footprint Precision Arduino Charlieplex:CRA04 -> Precision Arduino Charlieplex 1.1:CRA04
- R501, R502: footprint Precision Arduino Charlieplex:0603-RES -> Precision Arduino Charlieplex 1.1:0603-RES
- S429: footprint Precision Arduino Charlieplex:B3U-1100P -> Precision Arduino Charlieplex 1.1:B3U-1100P
- U401: footprint Precision Arduino Charlieplex:TQFP32-08 -> Precision Arduino Charlieplex 1.1:TQFP32-08
- U501: footprint Precision Arduino Charlieplex:SSOP28DB -> Precision Arduino Charlieplex 1.1:SSOP28DB
- U602: footprint Precision Arduino Charlieplex:SC-70-6 -> Precision Arduino Charlieplex 1.1:SC-70-6
- Y401: value 12.00 -> 16MHz; footprint Precision Arduino Charlieplex:CRYSTAL_SMD -> Precision Arduino Charlieplex 1.1:CRYSTAL_SMD
Connections:
- J3 pad 4: /D13 -> /P16
- J3 pad 6: /D11 -> /P01
- J5 pad 4: /D13 -> /P16
- J5 pad 6: /D11 -> /P01
- R606 pad 2: VCC -> (no net)
- R606 pad 3: VCC -> (no net)
- R606 pad 6: /D13 -> (no net)
- R606 pad 7: /D12 -> (no net)
- R606 pad 8: /D11 -> /D12
- U401 pad 15: /D11 -> /P01
- U401 pad 17: /D13 -> /P16
- U401 pad 19: /P01 -> Net-(U401-Pad19)
- U401 pad 22: /P16 -> Net-(U401-Pad22)
- U501 pad 17: Net-(U501-Pad17) -> /3V3
- U501 pad 26: Net-(U501-Pad26) -> GND
- U501 pad 5: /USB_RX -> /AT_TX
Routing:
- net GND: track 158.2 -> 0.00 mm, vias 4 -> 5
- net /D11: track 81.1 -> 0.00 mm, vias 2 -> 0
- net /D13: track 50.6 -> 0.00 mm, vias 2 -> 0
- net VCC: track 118.5 -> 77.2 mm
- net /AT_TX: track 64.1 -> 33.3 mm
- net /P16: track 43.2 -> 72.8 mm, vias 0 -> 1
- net /PPS: track 47.1 -> 18.1 mm, vias 2 -> 0
- net /P01: track 9.41 -> 35.8 mm, vias 0 -> 1
- net /3V3: track 0.00 -> 23.9 mm
- net /GPS_RX: track 22.5 -> 0.00 mm
- net /D12: track 73.2 -> 53.3 mm, vias 2 -> 3
- net /GPS_TX: track 45.5 -> 27.9 mm, vias 3 -> 2
- net /USB_TX: track 19.2 -> 7.39 mm, vias 4 -> 2
- net /USB_RX: track 11.6 -> 0.00 mm, vias 2 -> 0
- net Net-(R501-Pad1): track 7.79 -> 12.6 mm
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- added copper zone on B.Cu, net GND
- added copper zone on F.Cu, net GND
Other:
- rule pad_to_mask_clearance: 0.05 -> 0.051
- board text added: "13 Apr 2012"
- board text added: "3V3"
- board text added: "BAT"
- board text added: "PPS"
- board text added: "RX"
- board text added: "TX"
- board text removed: "7 Nov 2011"
